Commit message: 完整的仿真链路已经搭建好了，但是底盘的运动控制有点问题

File: urdfs/T002_description/xacro/T002_description.urdf.xacro (robot description, xacro)
@@ -1,125 +1,261 @@
 <?xml version="1.0"?>
-<robot xmlns:xacro="http://www.ros.org/wiki/xacro" name="T002_Neck">
-  <!-- ===== ros2_control hardware plugin ===== -->
+<robot xmlns:xacro="http://www.ros.org/wiki/xacro" name="T002_Robot">
   <xacro:include filename="$(find t002_description)/xacro/ros2control.xacro"/>
-  <xacro:property name="joints_config_file"
-    value="$(find t002_description)/xacro/joints_config.yaml"/>
-  <xacro:property name="imu_config_file"
-    value="$(find t002_description)/xacro/imu_config.yaml"/>
-  <xacro:t002_ros2_control
-    name="T002Hardware"
-    joints_config_file="${joints_config_file}"
-    imu_config_file="${imu_config_file}"/>
-  <!-- ===== base_link ===== -->
+  <xacro:property name="joints_config_file" value="$(find t002_description)/xacro/joints_config.yaml"/>
+  <xacro:property name="imu_config_file" value="$(find t002_description)/xacro/imu_config.yaml"/>
+  <xacro:t002_ros2_control name="T002Hardware" joints_config_file="${joints_config_file}" imu_config_file="${imu_config_file}"/>
   <link name="base_link">
     <inertial>
-      <origin xyz="0.055815 -0.057719 -0.10153" rpy="0 0 0"/>
-      <mass value="0.23606"/>
-      <inertia ixx="0.00015043" ixy="7.6217E-09" ixz="-3.8509E-08"
-               iyy="0.00027587" iyz="2.2368E-07" izz="0.00039725"/>
-    </inertial>
-    <visual>
-      <origin xyz="0 0 0" rpy="0 0 0"/>
-      <geometry>
-        <mesh filename="package://t002_description/meshes/base_link.STL"/>
-      </geometry>
-      <material name=""><color rgba="1 1 1 1"/></material>
-    </visual>
-    <collision>
-      <origin xyz="0 0 0" rpy="0 0 0"/>
-      <geometry>
-        <mesh filename="package://t002_description/meshes/base_link.STL"/>
-      </geometry>
-    </collision>
-  </link>
-  <!-- ===== Ylink ===== -->
-  <link name="Ylink">
-    <inertial>
-      <origin xyz="-0.0006989 0.010921 0.020993" rpy="0 0 0"/>
-      <mass value="0.17216"/>
-      <inertia ixx="0.00011989" ixy="5.0469E-08" ixz="1.0432E-06"
-               iyy="0.00011905" iyz="-1.6433E-05" izz="0.00013647"/>
-    </inertial>
-    <visual>
-      <origin xyz="0 0 0" rpy="0 0 0"/>
-      <geometry>
-        <mesh filename="package://t002_description/meshes/Ylink.STL"/>
-      </geometry>
-      <material name=""><color rgba="1 1 1 1"/></material>
-    </visual>
-    <collision>
-      <origin xyz="0 0 0" rpy="0 0 0"/>
-      <geometry>
-        <mesh filename="package://t002_description/meshes/Ylink.STL"/>
-      </geometry>
-    </collision>
-  </link>
-  <!-- ===== yaw joint ===== -->
-  <joint name="yaw" type="revolute">
-    <origin xyz="0.055826 -0.057765 -0.065609" rpy="0 0 0"/>
-    <parent link="base_link"/>
-    <child link="Ylink"/>
-    <axis xyz="0 0 1"/>
-    <limit lower="-3.14" upper="3.14" effort="10" velocity="10"/>
-  </joint>
-  <!-- ===== Plink ===== -->
-  <link name="Plink">
-    <inertial>
-      <origin xyz="-0.00060859 0.0094805 2.065E-08" rpy="0 0 0"/>
-      <mass value="0.0021745"/>
-      <inertia ixx="5.685E-08" ixy="-5.9793E-11" ixz="-1.5825E-23"
-               iyy="5.7771E-08" iyz="-6.2549E-24" izz="6.269E-08"/>
-    </inertial>
-    <visual>
-      <origin xyz="0 0 0" rpy="0 0 0"/>
-      <geometry>
-        <mesh filename="package://t002_description/meshes/Plink.STL"/>
-      </geometry>
-      <material name=""><color rgba="0.79216 0.81961 0.93333 1"/></material>
-    </visual>
-    <collision>
-      <origin xyz="0 0 0" rpy="0 0 0"/>
-      <geometry>
-        <mesh filename="package://t002_description/meshes/Plink.STL"/>
-      </geometry>
-    </collision>
-  </link>
-  <!-- ===== pitch joint ===== -->
-  <joint name="pitch" type="revolute">
-    <origin xyz="-0.001057 0.016466 0.07945" rpy="0 0 0"/>
-    <parent link="Ylink"/>
-    <child link="Plink"/>
-    <axis xyz="0.064062 -0.99795 0"/>
-    <limit lower="-0.35" upper="0.35" effort="10" velocity="10"/>
-  </joint>
-  <!-- ===== Rlink ===== -->
-  <link name="Rlink">
-    <inertial>
-      <origin xyz="0.0071042 -0.035816 0.11657" rpy="0 0 0"/>
-      <mass value="1.9595"/>
-      <inertia ixx="0.0039007" ixy="-0.0001003" ixz="-2.0935E-05"
-               iyy="0.0055561" iyz="9.9024E-05" izz="0.0058803"/>
-    </inertial>
-    <visual>
-      <origin xyz="0 0 0" rpy="0 0 0"/>
-      <geometry>
-        <mesh filename="package://t002_description/meshes/Rlink.STL"/>
-      </geometry>
-      <material name=""><color rgba="0.79216 0.81961 0.93333 1"/></material>
-    </visual>
-    <collision>
-      <origin xyz="0 0 0" rpy="0 0 0"/>
-      <geometry>
-        <mesh filename="package://t002_description/meshes/Rlink.STL"/>
-      </geometry>
-    </collision>
-  </link>
-  <!-- ===== row joint ===== -->
-  <joint name="roll" type="revolute">
-    <origin xyz="-0.0046004 0.0092242 0" rpy="0 0 0"/>
-    <parent link="Plink"/>
-    <child link="Rlink"/>
-    <axis xyz="-0.99795 -0.064062 0"/>
-    <limit lower="-0.35" upper="0.35" effort="10" velocity="10"/>
+      <origin xyz="-0.160245654377849 -0.245416001589025 0.0551986514208551" rpy="0 0 0" />
+      <mass value="3.14792391169408" />
+      <inertia ixx="0.00987479852585863" ixy="0.000272766373301422" ixz="-1.03799819068223E-07" iyy="0.0036482619483936" iyz="-2.77588089220767E-07" izz="0.0110220695530071" />
+    </inertial>
+    <visual>
+      <origin xyz="0 0 0" rpy="0 0 0" />
+      <geometry>
+        <mesh filename="package://t002_description/meshes/base_link.STL" />
+      </geometry>
+      <material name="">
+        <color rgba="0.898039215686275 0.917647058823529 0.929411764705882 1" />
+      </material>
+    </visual>
+    <collision>
+      <origin xyz="0 0 0" rpy="0 0 0" />
+      <geometry>
+        <mesh filename="package://t002_description/meshes/base_link.STL" />
+      </geometry>
+    </collision>
+  </link>
+  <link name="waist_Link">
+    <inertial>
+      <origin xyz="0.000758270795805954 -0.000624090558024759 0.117127000839056" rpy="0 0 0" />
+      <mass value="4.35472302636246" />
+      <inertia ixx="0.0144064319373154" ixy="0.000269396723106418" ixz="5.57166974523934E-07" iyy="0.014397542506614" iyz="-2.19849900866876E-06" izz="0.027237348766065" />
+    </inertial>
+    <visual>
+      <origin xyz="0 0 0" rpy="0 0 0" />
+      <geometry>
+        <mesh filename="package://t002_description/meshes/waist_Link.STL" />
+      </geometry>
+      <material name="">
+        <color rgba="0.752941176470588 0.752941176470588 0.752941176470588 1" />
+      </material>
+    </visual>
+    <collision>
+      <origin xyz="0 0 0" rpy="0 0 0" />
+      <geometry>
+        <mesh filename="package://t002_description/meshes/waist_Link.STL" />
+      </geometry>
+    </collision>
+  </link>
+  <joint name="waist_joint" type="revolute">
+    <origin xyz="-0.160242981103207 -0.245425719745925 0.146317082445813" rpy="0 0 0" />
+    <parent link="base_link" />
+    <child link="waist_Link" />
+    <axis xyz="0 0 1" />
+    <limit lower="-3.14" upper="3.14" effort="100" velocity="50" />
+  </joint>
+  <link name="neck_yaw_Link">
+    <inertial>
+      <origin xyz="-0.010896 2.1954E-06 0.02051" rpy="0 0 0" />
+      <mass value="0.17256" />
+      <inertia ixx="0.00011905" ixy="3.5567E-09" ixz="1.6466E-05" iyy="0.0001199" iyz="-1.1405E-08" izz="0.00013648" />
+    </inertial>
+    <visual>
+      <origin xyz="0 0 0" rpy="0 0 0" />
+      <geometry>
+        <mesh filename="package://t002_description/meshes/neck-yaw_Link.STL" />
+      </geometry>
+      <material name="">
+        <color rgba="0.75294 0.75294 0.75294 1" />
+      </material>
+    </visual>
+    <collision>
+      <origin xyz="0 0 0" rpy="0 0 0" />
+      <geometry>
+        <mesh filename="package://t002_description/meshes/neck-yaw_Link.STL" />
+      </geometry>
+    </collision>
+  </link>
+  <joint name="neck_yaw_joint" type="revolute">
+    <origin xyz="0 0 0.2155" rpy="0 0 2.3562" />
+    <parent link="waist_Link" />
+    <child link="neck_yaw_Link" />
+    <axis xyz="0 0 1" />
+    <limit lower="-3.14" upper="3.14" effort="100" velocity="50" />
+  </joint>
+  <link name="neck_pitch_Link">
+    <inertial>
+      <origin xyz="-1.17752753103773E-08 -8.19698281473435E-09 -0.00788903490226288" rpy="0 0 0" />
+      <mass value="0.00217444221491406" />
+      <inertia ixx="5.68460266068729E-08" ixy="8.23042191731768E-14" ixz="1.22567126147768E-13" iyy="6.26901436196879E-08" iyz="8.10191632139002E-14" izz="5.77744934902568E-08" />
+    </inertial>
+    <visual>
+      <origin xyz="0 0 0" rpy="0 0 0" />
+      <geometry>
+        <mesh filename="package://t002_description/meshes/neck-pitch_Link.STL" />
+      </geometry>
+      <material name="">
+        <color rgba="1 1 1 1" />
+      </material>
+    </visual>
+    <collision>
+      <origin xyz="0 0 0" rpy="0 0 0" />
+      <geometry>
+        <mesh filename="package://t002_description/meshes/neck-pitch_Link.STL" />
+      </geometry>
+    </collision>
+  </link>
+  <joint name="neck_pitch_joint" type="revolute">
+    <origin xyz="-0.018111 0 0.07895" rpy="1.5708 0 1.5708" />
+    <parent link="neck_yaw_Link" />
+    <child link="neck_pitch_Link" />
+    <axis xyz="0 0 1" />
+    <limit lower="-3.14" upper="3.14" effort="100" velocity="50" />
+  </joint>
+  <link name="neck_roll_Link">
+    <inertial>
+      <origin xyz="-0.00525257353130502 -0.0977894394825203 -0.00840762569658554" rpy="0 0 0" />
+      <mass value="0.937804199456253" />
+      <inertia ixx="0.00485714170217262" ixy="-0.00010054019285476" ixz="-1.95513043546368E-05" iyy="0.00518201961483246" iyz="-1.43697206549072E-05" izz="0.00382636692871019" />
+    </inertial>
+    <visual>
+      <origin xyz="0 0 0" rpy="0 0 0" />
+      <geometry>
+        <mesh filename="package://t002_description/meshes/neck-roll_Link.STL" />
+      </geometry>
+      <material name="">
+        <color rgba="1 1 1 1" />
+      </material>
+    </visual>
+    <collision>
+      <origin xyz="0 0 0" rpy="0 0 0" />
+      <geometry>
+        <mesh filename="package://t002_description/meshes/neck-roll_Link.STL" />
+      </geometry>
+    </collision>
+  </link>
+  <joint name="neck_roll_joint" type="revolute">
+    <origin xyz="-0.007889 0 -0.007889" rpy="1.5708 1.5708 -1.5944" />
+    <parent link="neck_pitch_Link" />
+    <child link="neck_roll_Link" />
+    <axis xyz="0 0 1" />
+    <limit lower="-3.14" upper="3.14" effort="100" velocity="50" />
+  </joint>
+  <link name="wheel_left_yaw_Link">
+    <inertial>
+      <origin xyz="0.00225102039641978 -0.00252527871050234 0.108109688229945" rpy="0 0 0" />
+      <mass value="0.610103997497279" />
+      <inertia ixx="0.000625154311267543" ixy="-0.000214617722534287" ixz="-2.2847996532257E-05" iyy="0.000625011994966997" iyz="-2.27954728208063E-05" izz="0.000550155090255592" />
+    </inertial>
+    <visual>
+      <origin xyz="0 0 0" rpy="0 0 0" />
+      <geometry>
+        <mesh filename="package://t002_description/meshes/wheel-left-yaw_Link.STL" />
+      </geometry>
+      <material name="">
+        <color rgba="1 1 1 1" />
+      </material>
+    </visual>
+    <collision>
+      <origin xyz="0 0 0" rpy="0 0 0" />
+      <geometry>
+        <mesh filename="package://t002_description/meshes/wheel-left-yaw_Link.STL" />
+      </geometry>
+    </collision>
+  </link>
+  <joint name="wheel_left_yaw_joint" type="revolute">
+    <origin xyz="-0.32024 -0.40043 0.097317" rpy="-3.1416 0 3.1416" />
+    <parent link="base_link" />
+    <child link="wheel_left_yaw_Link" />
+    <axis xyz="0 0 -1" />
+    <limit lower="-3.14" upper="3.14" effort="100" velocity="50" />
+  </joint>
+  <link name="wheel_left_roll_Link">
+    <inertial>
+      <origin xyz="-2.4980018054066E-16 -3.46944695195361E-18 -0.000122162402514281" rpy="0 0 0" />
+      <mass value="0.190107278624991" />
+      <inertia ixx="0.000268176883616176" ixy="-5.4580685538699E-20" ixz="-1.0842021724855E-19" iyy="0.000268176883616176" iyz="-1.07096728268466E-19" izz="0.000504675491907474" />
+    </inertial>
+    <visual>
+      <origin xyz="0 0 0" rpy="0 0 0" />
+      <geometry>
+        <mesh filename="package://t002_description/meshes/wheel-left-roll_Link.STL" />
+      </geometry>
+      <material name="">
+        <color rgba="1 1 1 1" />
+      </material>
+    </visual>
+    <collision>
+      <origin xyz="0 0 0" rpy="0 0 0" />
+      <geometry>
+        <mesh filename="package://t002_description/meshes/wheel-left-roll_Link.STL" />
+      </geometry>
+    </collision>
+  </link>
+  <joint name="wheel_left_roll_joint" type="revolute">
+    <origin xyz="-0.00136589935180897 0.00429095489768716 0.12851606406394" rpy="1.5707963267949 0.00659792478876605 0.785398163397464" />
+    <parent link="wheel_left_yaw_Link" />
+    <child link="wheel_left_roll_Link" />
+    <axis xyz="0 0 -1" />
+    <limit lower="-3.14" upper="3.14" effort="100" velocity="50" />
+  </joint>
+  <link name="wheel_right_yaw_Link">
+    <inertial>
+      <origin xyz="0 0 0" rpy="0 0 0" />
+      <mass value="0.610103997497279" />
+      <inertia ixx="0" ixy="0" ixz="0" iyy="0" iyz="0" izz="0" />
+    </inertial>
+    <visual>
+      <origin xyz="0 0 0" rpy="0 0 0" />
+      <geometry>
+        <mesh filename="package://t002_description/meshes/wheel-right-yaw_Link.STL" />
+      </geometry>
+      <material name="">
+        <color rgba="1 1 1 1" />
+      </material>
+    </visual>
+    <collision>
+      <origin xyz="0 0 0" rpy="0 0 0" />
+      <geometry>
+        <mesh filename="package://t002_description/meshes/wheel-right-yaw_Link.STL" />
+      </geometry>
+    </collision>
+  </link>
+  <joint name="wheel_right_yaw_joint" type="revolute">
+    <origin xyz="-0.000242981103206271 -0.0904257197459303 0.0973170824458125" rpy="-3.14159265358979 0 3.14159265358979" />
+    <parent link="base_link" />
+    <child link="wheel_right_yaw_Link" />
+    <axis xyz="0 0 -1" />
+    <limit lower="-3.14" upper="3.14" effort="100" velocity="50" />
+  </joint>
+  <link name="wheel_right_roll_Link">
+    <inertial>
+      <origin xyz="-2.28983498828939E-16 -3.46944695195361E-18 -0.00012216240251426" rpy="0 0 0" />
+      <mass value="0.190107278624991" />
+      <inertia ixx="0.000268176883616176" ixy="-1.11173074327127E-21" ixz="-8.13151629364128E-20" iyy="0.000268176883616176" iyz="-8.00975530747348E-20" izz="0.000504675491907474" />
+    </inertial>
+    <visual>
+      <origin xyz="0 0 0" rpy="0 0 0" />
+      <geometry>
+        <mesh filename="package://t002_description/meshes/wheel-right-roll_Link.STL" />
+      </geometry>
+      <material name="">
+        <color rgba="1 1 1 1" />
+      </material>
+    </visual>
+    <collision>
+      <origin xyz="0 0 0" rpy="0 0 0" />
+      <geometry>
+        <mesh filename="package://t002_description/meshes/wheel-right-roll_Link.STL" />
+      </geometry>
+    </collision>
+  </link>
+  <joint name="wheel_right_roll_joint" type="revolute">
+    <origin xyz="-0.00136589935180871 0.00429095489768724 0.12851606406394" rpy="1.5707963267949 0.00659792478876655 0.785398163397398" />
+    <parent link="wheel_right_yaw_Link" />
+    <child link="wheel_right_roll_Link" />
+    <axis xyz="0 0 1" />
+    <limit lower="-3.14" upper="3.14" effort="100" velocity="50" />
   </joint>
 </robot>

File: urdfs/T002_description/xacro/ros2control.xacro (robot description, xacro)
@@ -17,33 +17,14 @@
     </joint>
   </xacro:macro>
-  <xacro:macro name="t002_ros2_control_imu" params="imu">
-    <sensor name="${imu.name}">
-      <param name="interface">${imu.interface}</param>
-      <param name="interface_type">${imu.interface_type}</param>
-      <param name="imu_type">${imu.imu_type}</param>
-      <param name="baudrate">${imu.baudrate}</param>
-      <state_interface name="orientation.x"/>
-      <state_interface name="orientation.y"/>
-      <state_interface name="orientation.z"/>
-      <state_interface name="orientation.w"/>
-      <state_interface name="angular_velocity.x"/>
-      <state_interface name="angular_velocity.y"/>
-      <state_interface name="angular_velocity.z"/>
-      <state_interface name="linear_acceleration.x"/>
-      <state_interface name="linear_acceleration.y"/>
-      <state_interface name="linear_acceleration.z"/>
-    </sensor>
-  </xacro:macro>
   <xacro:macro name="t002_ros2_control" params="
       name:=T002Hardware
+      hardware_plugin:=robot_hardware/RobotHardwareNode
       joints_config_file:=joints_config.yaml
       imu_config_file:=imu_config.yaml">
     <xacro:property name="joints_config" value="${xacro.load_yaml(joints_config_file)}"/>
-    <xacro:property name="imu_config" value="${xacro.load_yaml(imu_config_file)}"/>
     <ros2_control name="${name}" type="system">
       <hardware>
-        <plugin>robot_hardware/RobotHardwareNode</plugin>
+        <plugin>${hardware_plugin}</plugin>
       </hardware>
-      <!-- 动态关节数 -->
       <xacro:if value="${len(joints_config['joints']) > 0}">
         <xacro:t002_ros2_control_joint joint="${joints_config['joints'][0]}"/>
@@ -55,7 +36,18 @@
         <xacro:t002_ros2_control_joint joint="${joints_config['joints'][2]}"/>
       </xacro:if>
-      <!-- 动态IMU -->
-      <xacro:if value="${imu_config['imus'] and len(imu_config['imus']) > 0}">
-        <xacro:t002_ros2_control_imu imu="${imu_config['imus'][0]}"/>
+      <xacro:if value="${len(joints_config['joints']) > 3}">
+        <xacro:t002_ros2_control_joint joint="${joints_config['joints'][3]}"/>
+      </xacro:if>
+      <xacro:if value="${len(joints_config['joints']) > 4}">
+        <xacro:t002_ros2_control_joint joint="${joints_config['joints'][4]}"/>
+      </xacro:if>
+      <xacro:if value="${len(joints_config['joints']) > 5}">
+        <xacro:t002_ros2_control_joint joint="${joints_config['joints'][5]}"/>
+      </xacro:if>
+      <xacro:if value="${len(joints_config['joints']) > 6}">
+        <xacro:t002_ros2_control_joint joint="${joints_config['joints'][6]}"/>
+      </xacro:if>
+      <xacro:if value="${len(joints_config['joints']) > 7}">
+        <xacro:t002_ros2_control_joint joint="${joints_config['joints'][7]}"/>
       </xacro:if>
     </ros2_control>
