Commit message: 脖子部分基本调试通了，然后仿真没有什么问题，准备接入摄像头

File: urdfs/T002_description/xacro/T002_gazebo_des.urdf.xacro (robot description, xacro)
@@ -265,3 +265,25 @@
     </plugin>
   </gazebo>
+  <link name="imu_link">
+      <visual>
+      <origin xyz="0 0 0.0" rpy="0 0 0"/>
+      <geometry>
+            <box size="0.02 0.02 0.02"/>
+      </geometry>
+    </visual>
+  </link>
+  <!-- imu joint -->
+  <joint name="imu_joint" type="fixed">
+      <parent link="waist_Link" />
+      <child link="imu_link" />
+      <origin xyz="0 0 0.02" />
+  </joint>
+      <gazebo reference="imu_link">
+      <sensor name="imu_sensor" type="imu">
+        <always_on>true</always_on>
+        <update_rate>100</update_rate>
+        <topic>/imu</topic>
+        <visualize>true</visualize>
+      </sensor>
+    </gazebo>
 </robot>
